File: IKEA-Samtid_LED-disk.sch (KiCad schematic (older format))
At the start: 0 parts

Commit message: Made schematic + placing a couple of LEDs.
Parts:
- added C1, C3: 100nF, symbol C
- added C2: 1µF, symbol C
- added C4: DNP, symbol C
- added DS1: 6A, symbol DIODESCH
- added F1, F2: 2A-poly, symbol FUSE
- added IC1: ATMEGA168PA-A, TQFP32, symbol ATMEGA168PA-A
- added JP1: AVR_ISP, symbol MADW__AVR_ISP
- added P1: FTDI, symbol CONN_6
- added P2: POWER, symbol CONN_2
- added R1: 10k, symbol R
Connections:
- new net: C3.1, IC1.20 (AREF)
- new net: F1.1, F2.1, P2.1 (P1)
- new net: DS1.1 (A), F1.2, F2.2
- new net +5V: C1.1, C2.1, DS1.2 (C), IC1.18 (AVCC), IC1.4 (VCC), IC1.6 (VCC), JP1.2 (VTG), P1.3, R1.2
- new net DTR: C4.1, C4.2, IC1.29 ((PCINT14/~RESET~)PC6), JP1.5 (RST), P1.6, R1.1
- new net GND: C1.2, C2.2, C3.2, IC1.21 (GND), IC1.3 (GND), IC1.5 (GND), JP1.6 (GND), P1.1, P2.2 (PM)
- new net LED_D: IC1.1 ((PCINT19/OC2B/INT1)PD3)
- new net MISO: IC1.16 ((PCINT4/MISO)PB4), JP1.1 (MISO)
- new net MOSI: IC1.15 ((PCINT3/OC2A/MOSI)PB3), JP1.4 (MOSI)
- new net RXI: IC1.30 ((PCINT16/RXD)PD0), P1.4
- new net SCK: IC1.17 ((PCINT5/SCK)PB5), JP1.3 (SCK)
- new net TXO: IC1.31 ((PCINT17/TXD)PD1), P1.5
- new net XTAL1: IC1.7 ((PCINT6/XTAL1/TOSC1)PB6)
- new net XTAL2: IC1.8 ((PCINT7/XTAL2/TOSC2)PB7)
- no-connect marks 0 -> 19
Other:
- note added: "WS2812B LEDs + capacitors"
