File: IKEA-Samtid_LED-disk.kicad_pcb (KiCad board)
At the start: 2 copper layers, 100 x 100 mm, 137 parts, among them IC1 ATMEGA168PA-A, P1 FTDI, P2 POWER

Commit message: Tracks...
Parts:
- C41, C42, C43, C44, C45, C46, C47, LED42, LED43: moved to B.Cu
- moved C41 190.9 mm to (176.8, 68.3), turned to 135 degrees
- moved C42 183.7 mm to (181.5, 74.1), turned to 123.8 degrees
- moved C43 173.4 mm to (184.9, 80.6), turned to 112.5 degrees
- moved C44 166.8 mm to (187.1, 87.6), turned to 101.2 degrees
- moved C45 155.1 mm to (187.8, 95.0), turned to 90 degrees
- moved C46 153.7 mm to (187.1, 102.4), turned to 78.7 degrees
- moved C47 141.3 mm to (184.9, 109.5), turned to 67.5 degrees
- moved LED42 127.7 mm to (194.1, 103.9), turned to 348.7 degrees
- moved LED43 118.5 mm to (191.6, 112.2), turned to 337.5 degrees
- moved C15 88.1 mm to (184.9, 109.5), turned to 67.4 degrees
- moved C14 83.4 mm to (187.1, 102.4), turned to 78.7 degrees
- moved LED11 17.9 mm to (191.6, 112.2), turned to 157.4 degrees
- moved LED10 15.3 mm to (194.1, 103.9), turned to 168.7 degrees
- moved C11 0.36 mm to (184.9, 80.6)
- moved C10 0.28 mm to (181.5, 74.1)
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Routing:
- net +5V: track 152.4 -> 278.9 mm, vias 5 -> 12
- net GND: track 185.3 -> 281.4 mm, vias 5 -> 12
- net Net-(LED41-Pad2): track 0.00 -> 13.1 mm
- net Net-(LED42-Pad2): track 0.00 -> 12.7 mm
- net Net-(LED5-Pad2): track 6.79 -> 8.84 mm
- net Net-(LED7-Pad2): track 6.87 -> 8.46 mm
- net /WS2812B-LEDs-1/A_OUT: track 6.93 -> 8.36 mm
- net Net-(LED6-Pad2): track 6.68 -> 7.47 mm

Commit message: Stuff.
Parts:
- moved LED22 275.1 mm to (-170.4, 133.9)
- moved LED21 264.3 mm to (-154.0, 144.0)
- moved LED20 262.4 mm to (-144.6, 154.7)
- moved LED19 261.3 mm to (-134.8, 169.5)
- moved LED18 258.3 mm to (-123.9, 173.7)
- moved LED16 253.9 mm to (-102.3, 168.1)
- moved LED17 253.7 mm to (-111.8, 169.0)
- moved LED15 246.6 mm to (-83.8, 180.0)
- moved LED14 239.0 mm to (-66.4, 177.3)
- moved LED13 235.8 mm to (-56.0, 166.2)
- moved C1 220.2 mm to (-33.8, 199.9)
- moved C2 220.2 mm to (-26.5, 199.7)
- moved C3 220.2 mm to (-33.8, 206.3)
- moved C4 220.2 mm to (-20.7, 192.3)
- moved JP1 220.2 mm to (-40.6, 201.8)
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
Commit message: This is getting very tedious.
Parts:
- C48, C49, C50, C51, C52, C66, C67, LED44, LED45, LED46, LED47, LED48, LED62, LED63: moved to B.Cu
- moved LED16 251.6 mm to (147.9, 142.0), turned to 90 degrees
- moved LED15 247.0 mm to (160.0, 140.6), turned to 112.5 degrees
- moved LED13 241.0 mm to (181.8, 126.8), turned to 135.1 degrees
- moved LED14 240.2 mm to (170.4, 137.2), turned to 112.5 degrees
- moved LED62 225.2 mm to (125.0, 57.6), turned to 123.8 degrees
- moved C35 214.2 mm to (135.5, 60.1), turned to 202.5 degrees
- moved C34 210.4 mm to (129.0, 63.6), turned to 213.8 degrees
- moved C66 207.2 mm to (129.0, 63.6), turned to 213.8 degrees
- moved LED63 205.9 mm to (132.8, 53.4), turned to 112.5 degrees
- moved C67 203.9 mm to (135.5, 60.1), turned to 202.5 degrees
- moved C18 183.8 mm to (167.5, 130.1), turned to 22.5 degrees
- moved C17 182.0 mm to (176.7, 121.7), turned to 45.1 degrees
- moved C16 170.9 mm to (181.4, 116.0), turned to 56.2 degrees
- moved LED12 163.3 mm to (187.4, 120.0), turned to 146.3 degrees
- moved LED30 156.2 mm to (125.0, 57.6), turned to 303.8 degrees
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Routing:
- net GND: track 281.4 -> 329.0 mm, vias 12 -> 14
- net +5V: track 278.9 -> 325.6 mm, vias 12 -> 14
- net Net-(LED62-Pad2): track 0.00 -> 13.3 mm
- net Net-(LED63-Pad2): track 0.00 -> 13.3 mm
- net Net-(LED30-Pad2): track 0.00 -> 7.46 mm, vias 0 -> 2
- net Net-(LED31-Pad2): track 0.00 -> 7.42 mm, vias 0 -> 2
