File: WS2812B-LEDs-2.sch (KiCad schematic (older format))
At the start: 64 parts

Commit message: Getting lost in hirarchical schematic sheets...
Connections:
- net +5V: no longer C37.1, C38.1, C39.1, C40.1, C41.1, C42.1, C43.1, C44.1, C45.1, C46.1, C47.1, C48.1, C49.1, C50.1, C51.1, C52.1, C53.1, C54.1, C55.1, C56.1, C57.1, C58.1, C59.1, C60.1, C61.1, C62.1, C63.1, C64.1, C65.1, C66.1, C67.1, C68.1, LED33.1 (VCC), LED34.1 (VCC), LED35.1 (VCC), LED36.1 (VCC), LED37.1 (VCC), LED38.1 (VCC), LED39.1 (VCC), LED40.1 (VCC), LED41.1 (VCC), LED42.1 (VCC), LED43.1 (VCC), LED44.1 (VCC), LED45.1 (VCC), LED46.1 (VCC), LED47.1 (VCC), LED48.1 (VCC), LED49.1 (VCC), LED50.1 (VCC), LED51.1 (VCC), LED52.1 (VCC), LED53.1 (VCC), LED54.1 (VCC), LED55.1 (VCC), LED57.1 (VCC), LED58.1 (VCC)
- net GND: no longer LED33.3 (GND), LED34.3 (GND), LED35.3 (GND), LED36.3 (GND), LED37.3 (GND), LED38.3 (GND), LED39.3 (GND), LED40.3 (GND), LED41.3 (GND), LED42.3 (GND), LED43.3 (GND), LED44.3 (GND), LED45.3 (GND), LED46.3 (GND), LED47.3 (GND), LED48.3 (GND), LED49.3 (GND), LED50.3 (GND), LED51.3 (GND), LED52.3 (GND)
- new net VCC: C37.1, C38.1, C39.1, C40.1, C41.1, C42.1, C43.1, C44.1, C45.1, C46.1, C47.1, C48.1, C49.1, C50.1, C51.1, C52.1, C53.1, C54.1, C55.1, C56.1, C57.1, C58.1, C59.1, C60.1, C61.1, C62.1, C63.1, C64.1, C65.1, C66.1, C67.1, C68.1

Commit message: Hirarchical schem. sheets have 'interesting' effects on net-names.
Connections:
- net +5V is gone; now on net VCC: LED56.1 (VCC), LED59.1 (VCC), LED60.1 (VCC), LED61.1 (VCC), LED62.1 (VCC), LED63.1 (VCC), LED64.1 (VCC)
- net GND: now also LED33.3 (GND), LED34.3 (GND), LED35.3 (GND), LED36.3 (GND), LED37.3 (GND), LED38.3 (GND), LED39.3 (GND), LED40.3 (GND), LED41.3 (GND), LED42.3 (GND), LED43.3 (GND), LED44.3 (GND), LED45.3 (GND), LED46.3 (GND), LED47.3 (GND), LED48.3 (GND), LED49.3 (GND), LED50.3 (GND), LED51.3 (GND), LED52.3 (GND)
- net VCC: now also LED33.1 (VCC), LED34.1 (VCC), LED35.1 (VCC), LED36.1 (VCC), LED37.1 (VCC), LED38.1 (VCC), LED39.1 (VCC), LED40.1 (VCC), LED41.1 (VCC), LED42.1 (VCC), LED43.1 (VCC), LED44.1 (VCC), LED45.1 (VCC), LED46.1 (VCC), LED47.1 (VCC), LED48.1 (VCC), LED49.1 (VCC), LED50.1 (VCC), LED51.1 (VCC), LED52.1 (VCC), LED53.1 (VCC), LED54.1 (VCC), LED55.1 (VCC), LED57.1 (VCC), LED58.1 (VCC)

Commit message: Being creative...
Parts:
- C37, C38, C39, C40, C41, C42, C43, C44, C45, C46, C47, C48, C49, C50, C51, C52, C53, C54, C55, C56, C57, C58, C59, C60, C61, C62, C63, C64, C65, C66, C67, C68: footprint (none) -> my_parts:MADW__C0805
- LED33, LED34, LED35, LED36, LED37, LED38, LED39, LED40, LED41, LED42, LED43, LED44, LED45, LED46, LED47, LED48, LED49, LED50, LED51, LED52, LED53, LED54, LED55, LED56, LED57, LED58, LED59, LED60, LED61, LED62, LED63, LED64: footprint (none) -> WS2812B:WS2812B_data-bridgeable

Commit message: Some cleanup. Still need to fix the power connector(s).
Parts:
- C37, C38, C39, C40, C41, C42, C43, C44, C45, C46, C47, C48, C49, C50, C51, C52, C53, C54, C55, C56, C57, C58, C59, C60, C61, C62, C63, C64, C65, C66, C67, C68: value C -> 1µF
Changed lines of the file:
@@
 P 7250 950
 F 0 "C37" H 7250 1050 40  0000 L CNN
-F 1 "C" H 7256 865 40  0000 L CNN
+F 1 "1µF" H 7256 865 40  0000 L CNN
 F 2 "my_parts:MADW__C0805" H 7288 800 30  0001 C CNN
 F 3 "" H 7250 950 60  0000 C CNN
@@
 P 7500 950
 F 0 "C39" H 7500 1050 40  0000 L CNN
-F 1 "C" H 7506 865 40  0000 L CNN
+F 1 "1µF" H 7506 865 40  0000 L CNN
 F 2 "my_parts:MADW__C0805" H 7538 800 30  0001 C CNN
 F 3 "" H 7500 950 60  0000 C CNN
@@
 P 7750 950
 F 0 "C41" H 7750 1050 40  0000 L CNN
-F 1 "C" H 7756 865 40  0000 L CNN
+F 1 "1µF" H 7756 865 40  0000 L CNN
 F 2 "my_parts:MADW__C0805" H 7788 800 30  0001 C CNN
 F 3 "" H 7750 950 60  0000 C CNN
@@
 P 8000 950
 F 0 "C43" H 8000 1050 40  0000 L CNN
-F 1 "C" H 8006 865 40  0000 L CNN
+F 1 "1µF" H 8006 865 40  0000 L CNN
 F 2 "my_parts:MADW__C0805" H 8038 800 30  0001 C CNN
 F 3 "" H 8000 950 60  0000 C CNN
@@
 P 8250 950
 F 0 "C45" H 8250 1050 40  0000 L CNN
-F 1 "C" H 8256 865 40  0000 L CNN
+F 1 "1µF" H 8256 865 40  0000 L CNN
 F 2 "my_parts:MADW__C0805" H 8288 800 30  0001 C CNN
 F 3 "" H 8250 950 60  0000 C CNN
@@
 P 8500 950
 F 0 "C47" H 8500 1050 40  0000 L CNN
-F 1 "C" H 8506 865 40  0000 L CNN
+F 1 "1µF" H 8506 865 40  0000 L CNN
 F 2 "my_parts:MADW__C0805" H 8538 800 30  0001 C CNN
 F 3 "" H 8500 950 60  0000 C CNN
@@
 P 8750 950
 F 0 "C49" H 8750 1050 40  0000 L CNN
-F 1 "C" H 8756 865 40  0000 L CNN
+F 1 "1µF" H 8756 865 40  0000 L CNN
 F 2 "my_parts:MADW__C0805" H 8788 800 30  0001 C CNN
 F 3 "" H 8750 950 60  0000 C CNN
@@
 P 9000 950
 F 0 "C51" H 9000 1050 40  0000 L CNN
-F 1 "C" H 9006 865 40  0000 L CNN
+F 1 "1µF" H 9006 865 40  0000 L CNN
 F 2 "my_parts:MADW__C0805" H 9038 800 30  0001 C CNN
 F 3 "" H 9000 950 60  0000 C CNN
@@
 P 9250 950
 F 0 "C53" H 9250 1050 40  0000 L CNN
-F 1 "C" H 9256 865 40  0000 L CNN
+F 1 "1µF" H 9256 865 40  0000 L CNN
 F 2 "my_parts:MADW__C0805" H 9288 800 30  0001 C CNN
 F 3 "" H 9250 950 60  0000 C CNN
@@
 P 9500 950
 F 0 "C55" H 9500 1050 40  0000 L CNN
-F 1 "C" H 9506 865 40  0000 L CNN
+F 1 "1µF" H 9506 865 40  0000 L CNN
 F 2 "my_parts:MADW__C0805" H 9538 800 30  0001 C CNN
 F 3 "" H 9500 950 60  0000 C CNN
@@
 P 9750 950
 F 0 "C57" H 9750 1050 40  0000 L CNN
-F 1 "C" H 9756 865 40  0000 L CNN
+F 1 "1µF" H 9756 865 40  0000 L CNN
 F 2 "my_parts:MADW__C0805" H 9788 800 30  0001 C CNN
 F 3 "" H 9750 950 60  0000 C CNN
@@
 P 10000 950
 F 0 "C59" H 10000 1050 40  0000 L CNN
-F 1 "C" H 10006 865 40  0000 L CNN
+F 1 "1µF" H 10006 865 40  0000 L CNN
 F 2 "my_parts:MADW__C0805" H 10038 800 30  0001 C CNN
 F 3 "" H 10000 950 60  0000 C CNN
@@
 P 10250 950
 F 0 "C61" H 10250 1050 40  0000 L CNN
-F 1 "C" H 10256 865 40  0000 L CNN
+F 1 "1µF" H 10256 865 40  0000 L CNN
 F 2 "my_parts:MADW__C0805" H 10288 800 30  0001 C CNN
 F 3 "" H 10250 950 60  0000 C CNN
@@
 P 10500 950
 F 0 "C63" H 10500 1050 40  0000 L CNN
-F 1 "C" H 10506 865 40  0000 L CNN
+F 1 "1µF" H 10506 865 40  0000 L CNN
 F 2 "my_parts:MADW__C0805" H 10538 800 30  0001 C CNN
 F 3 "" H 10500 950 60  0000 C CNN
@@
 P 10750 950
 F 0 "C65" H 10750 1050 40  0000 L CNN
-F 1 "C" H 10756 865 40  0000 L CNN
+F 1 "1µF" H 10756 865 40  0000 L CNN
 F 2 "my_parts:MADW__C0805" H 10788 800 30  0001 C CNN
 F 3 "" H 10750 950 60  0000 C CNN
@@
 P 11000 950
 F 0 "C67" H 11000 1050 40  0000 L CNN
-F 1 "C" H 11006 865 40  0000 L CNN
+F 1 "1µF" H 11006 865 40  0000 L CNN
 F 2 "my_parts:MADW__C0805" H 11038 800 30  0001 C CNN
 F 3 "" H 11000 950 60  0000 C CNN
@@
 P 7250 1800
 F 0 "C38" H 7250 1900 40  0000 L CNN
-F 1 "C" H 7256 1715 40  0000 L CNN
+F 1 "1µF" H 7256 1715 40  0000 L CNN
 F 2 "my_parts:MADW__C0805" H 7288 1650 30  0001 C CNN
 F 3 "" H 7250 1800 60  0000 C CNN
@@
 P 7500 1800
 F 0 "C40" H 7500 1900 40  0000 L CNN
-F 1 "C" H 7506 1715 40  0000 L CNN
+F 1 "1µF" H 7506 1715 40  0000 L CNN
 F 2 "my_parts:MADW__C0805" H 7538 1650 30  0001 C CNN
 F 3 "" H 7500 1800 60  0000 C CNN
@@
 P 7750 1800
 F 0 "C42" H 7750 1900 40  0000 L CNN
-F 1 "C" H 7756 1715 40  0000 L CNN
+F 1 "1µF" H 7756 1715 40  0000 L CNN
 F 2 "my_parts:MADW__C0805" H 7788 1650 30  0001 C CNN
 F 3 "" H 7750 1800 60  0000 C CNN
@@
 P 8000 1800
 F 0 "C44" H 8000 1900 40  0000 L CNN
-F 1 "C" H 8006 1715 40  0000 L CNN
+F 1 "1µF" H 8006 1715 40  0000 L CNN
 F 2 "my_parts:MADW__C0805" H 8038 1650 30  0001 C CNN
 F 3 "" H 8000 1800 60  0000 C CNN
@@
 P 8250 1800
 F 0 "C46" H 8250 1900 40  0000 L CNN
-F 1 "C" H 8256 1715 40  0000 L CNN
+F 1 "1µF" H 8256 1715 40  0000 L CNN
 F 2 "my_parts:MADW__C0805" H 8288 1650 30  0001 C CNN
 F 3 "" H 8250 1800 60  0000 C CNN
@@
 P 8500 1800
 F 0 "C48" H 8500 1900 40  0000 L CNN
-F 1 "C" H 8506 1715 40  0000 L CNN
+F 1 "1µF" H 8506 1715 40  0000 L CNN
 F 2 "my_parts:MADW__C0805" H 8538 1650 30  0001 C CNN
 F 3 "" H 8500 1800 60  0000 C CNN
@@
 P 8750 1800
 F 0 "C50" H 8750 1900 40  0000 L CNN
-F 1 "C" H 8756 1715 40  0000 L CNN
+F 1 "1µF" H 8756 1715 40  0000 L CNN
 F 2 "my_parts:MADW__C0805" H 8788 1650 30  0001 C CNN
 F 3 "" H 8750 1800 60  0000 C CNN
@@
 P 9000 1800
 F 0 "C52" H 9000 1900 40  0000 L CNN
-F 1 "C" H 9006 1715 40  0000 L CNN
+F 1 "1µF" H 9006 1715 40  0000 L CNN
 F 2 "my_parts:MADW__C0805" H 9038 1650 30  0001 C CNN
 F 3 "" H 9000 1800 60  0000 C CNN
@@
 P 9250 1800
 F 0 "C54" H 9250 1900 40  0000 L CNN
-F 1 "C" H 9256 1715 40  0000 L CNN
+F 1 "1µF" H 9256 1715 40  0000 L CNN
 F 2 "my_parts:MADW__C0805" H 9288 1650 30  0001 C CNN
 F 3 "" H 9250 1800 60  0000 C CNN
@@
 P 9500 1800
 F 0 "C56" H 9500 1900 40  0000 L CNN
-F 1 "C" H 9506 1715 40  0000 L CNN
+F 1 "1µF" H 9506 1715 40  0000 L CNN
 F 2 "my_parts:MADW__C0805" H 9538 1650 30  0001 C CNN
 F 3 "" H 9500 1800 60  0000 C CNN
@@
 P 9750 1800
 F 0 "C58" H 9750 1900 40  0000 L CNN
-F 1 "C" H 9756 1715 40  0000 L CNN
+F 1 "1µF" H 9756 1715 40  0000 L CNN
 F 2 "my_parts:MADW__C0805" H 9788 1650 30  0001 C CNN
 F 3 "" H 9750 1800 60  0000 C CNN
@@
 P 10000 1800
 F 0 "C60" H 10000 1900 40  0000 L CNN
-F 1 "C" H 10006 1715 40  0000 L CNN
+F 1 "1µF" H 10006 1715 40  0000 L CNN
 F 2 "my_parts:MADW__C0805" H 10038 1650 30  0001 C CNN
 F 3 "" H 10000 1800 60  0000 C CNN
@@
 P 10250 1800
 F 0 "C62" H 10250 1900 40  0000 L CNN
-F 1 "C" H 10256 1715 40  0000 L CNN
+F 1 "1µF" H 10256 1715 40  0000 L CNN
 F 2 "my_parts:MADW__C0805" H 10288 1650 30  0001 C CNN
 F 3 "" H 10250 1800 60  0000 C CNN
@@
 P 10500 1800
 F 0 "C64" H 10500 1900 40  0000 L CNN
-F 1 "C" H 10506 1715 40  0000 L CNN
+F 1 "1µF" H 10506 1715 40  0000 L CNN
 F 2 "my_parts:MADW__C0805" H 10538 1650 30  0001 C CNN
 F 3 "" H 10500 1800 60  0000 C CNN
@@
 P 10750 1800
 F 0 "C66" H 10750 1900 40  0000 L CNN
-F 1 "C" H 10756 1715 40  0000 L CNN
+F 1 "1µF" H 10756 1715 40  0000 L CNN
 F 2 "my_parts:MADW__C0805" H 10788 1650 30  0001 C CNN
 F 3 "" H 10750 1800 60  0000 C CNN
@@
 P 11000 1800
 F 0 "C68" H 11000 1900 40  0000 L CNN
-F 1 "C" H 11006 1715 40  0000 L CNN
+F 1 "1µF" H 11006 1715 40  0000 L CNN
 F 2 "my_parts:MADW__C0805" H 11038 1650 30  0001 C CNN
 F 3 "" H 11000 1800 60  0000 C CNN
