File: IKEA-Samtid_mood-light_esp8266-adapter.sch (KiCad schematic (older format))
At the start: 5 parts, among them P1 ESP8266, P2 mood-light, U1 AMS1117-3.3

Commit message: ESP8266 adapter board reduced in size.
Parts:
- removed P1: ESP8266, DIL-Headers:DIL-4, symbol CONN_4X2
- added P1: ESP8266-01, DIL-Headers:DIL-4, symbol ESP8266-01
- added R1, R2, R3, R4: 10k, my_parts:MADW__R0603_2, symbol R
Connections:
- wire segments 25 -> 38
- no-connect marks 2 -> 0
Other:
- moved on the sheet: C1, C2, P2, U1

Commit message: ESP8266 adapter: changed RX/TX netnames to avoid confusion.
Connections:
- net RXI: now also P1.1 (RXI), P2.5; no longer P1.8 (TXO), P2.4
- net TXO: now also P1.8 (TXO), P2.4; no longer P1.1 (RXI), P2.5
Changed lines of the file:
@@
 Sheet 1 1
 Title "IKEA-Samtid_mood-light_esp8266-adapter"
-Date "Thu 12 Mar 2015"
-Rev "0.2"
+Date "Fri 13 Mar 2015"
+Rev "0.3"
 Comp "2015 - blog.spitzenpfeil.org"
 Comment1 ""
@@
 $EndComp
 Text Label 4100 4250 2    60   ~ 0
+TXO
+Text Label 4100 4150 2    60   ~ 0
 RXI
-Text Label 4100 4150 2    60   ~ 0
-TXO
 $Comp
 L GND #PWR02
@@
 	4200 4850 4250 4850
 Text Label 5800 4700 0    60   ~ 0
+RXI
+Text Label 5800 4600 0    60   ~ 0
 TXO
-Text Label 5800 4600 0    60   ~ 0
-RXI
 Text Label 5800 4300 0    60   ~ 0
 RST
